File: pc6001-meanwell-psu-adapter.kicad_pcb (KiCad board)
At the start: 2 copper layers, 195 x 84 mm, 5 parts, among them J1 Meanwell RPT-60B PSU module

Commit message: Better explainers
Other:
- board text added: "+12V"
- board text added: "+5V"
- board text added: "-12V"
- board text added: "GND"
- board text added: "Housing"
- board text added: "JST VHR"
- board text added: "L"
- board text added: "N"
- board text added: "SVH-21T-P1.1"
- board text added: "Terminals"
Changed lines of the file:
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@@
+	)
+	(gr_line
+		(start 81.28 107.315)
+		(end 70.485 107.315)
+		(stroke
+			(width 0.15)
+			(type default)
+		)
+		(layer "F.SilkS")
+	)
+	(gr_line
+		(start 95.25 107.315)
+		(end 70.485 107.315)
+		(stroke
+			(width 0.15)
+			(type default)
+		)
+		(layer "F.SilkS")
+	)
+	(gr_line
+		(start 70.485 110.49)
+		(end 95.25 110.49)
+		(stroke
+			(width 0.15)
+			(type default)
+		)
+		(layer "F.SilkS")
+	)
+	(gr_line
+		(start 95.25 107.315)
+		(end 95.25 113.665)
+		(stroke
+			(width 0.15)
+			(type default)
+		)
+		(layer "F.SilkS")
+	)
+	(gr_line
+		(start 81.28 113.665)
+		(end 81.28 107.315)
+		(stroke
+			(width 0.15)
+			(type default)
+		)
+		(layer "F.SilkS")
+	)
+	(gr_line
+		(start 70.485 113.665)
+		(end 70.485 107.315)
+		(stroke
+			(width 0.15)
+			(type default)
+		)
+		(layer "F.SilkS")
+	)
+	(gr_line
+		(start 70.485 113.665)
+		(end 95.25 113.665)
+		(stroke
+			(width 0.15)
+			(type default)
+		)
+		(layer "F.SilkS")
 	)
 	(gr_line
@@
 		(layer "Edge.Cuts")
 	)
+	(gr_text "JST VHR"
+		(at 88.646 109.855 0)
+		(layer "F.SilkS")
+		(effects
+			(font
+				(size 1 1)
+				(thickness 0.15)
+			)
+			(justify bottom)
+		)
+	)
+	(gr_text "+12V"
+		(at 103.505 80.645 0)
+		(layer "F.SilkS")
+		(effects
+			(font
+				(size 1 1)
+				(thickness 0.15)
+			)
+			(justify left bottom)
+		)
+	)
 	(gr_text "Attach safety ground with ring terminal to chassis"
 		(at 118.745 114.935 0)
@@
 			)
 			(justify right top)
+		)
+	)
+	(gr_text "+5V"
+		(at 103.505 90.805 0)
+		(layer "F.SilkS")
+		(effects
+			(font
+				(size 1 1)
+				(thickness 0.15)
+			)
+			(justify left bottom)
+		)
+	)
+	(gr_text "Terminals"
+		(at 76.2 113.03 0)
+		(layer "F.SilkS")
+		(effects
+			(font
+				(size 1 1)
+				(thickness 0.2)
+				(bold yes)
+			)
+			(justify bottom)
+		)
+	)
+	(gr_text "GND"
+		(at 103.505 85.725 0)
+		(layer "F.SilkS")
+		(effects
+			(font
+				(size 1 1)
+				(thickness 0.15)
+			)
+			(justify left bottom)
+		)
+	)
+	(gr_text "L"
+		(at 215.265 103.505 0)
+		(layer "F.SilkS")
+		(effects
+			(font
+				(size 1 1)
+				(thickness 0.15)
+			)
+			(justify left bottom)
+		)
+	)
+	(gr_text "Housing"
+		(at 76.2 109.855 0)
+		(layer "F.SilkS")
+		(effects
+			(font
+				(size 1 1)
+				(thickness 0.2)
+				(bold yes)
+			)
+			(justify bottom)
 		)
 	)
@@
 		)
 	)
+	(gr_text "GND"
+		(at 103.505 83.185 0)
+		(layer "F.SilkS")
+		(effects
+			(font
+				(size 1 1)
+				(thickness 0.15)
+			)
+			(justify left bottom)
+		)
+	)
+	(gr_text "N"
+		(at 215.265 93.98 0)
+		(layer "F.SilkS")
+		(effects
+			(font
+				(size 1 1)
+				(thickness 0.15)
+			)
+			(justify left bottom)
+		)
+	)
+	(gr_text "-12V"
+		(at 103.505 78.105 0)
+		(layer "F.SilkS")
+		(effects
+			(font
+				(size 1 1)
+				(thickness 0.15)
+			)
+			(justify left bottom)
+		)
+	)
+	(gr_text "SVH-21T-P1.1"
+		(at 82.804 113.03 0)
+		(layer "F.SilkS")
+		(effects
+			(font
+				(size 1 1)
+				(thickness 0.15)
+			)
+			(justify left bottom)
+		)
+	)
+	(gr_text "+5V"
+		(at 103.505 88.265 0)
+		(layer "F.SilkS")
+		(effects
+			(font
+				(size 1 1)
+				(thickness 0.15)
+			)
+			(justify left bottom)
+		)
+	)

Commit message: M4 holes - untested
Parts:
- removed the REF** at (56.8, 54.8)
- removed the REF** at (56.8, 129.2)
- removed the REF** at (231.0, 129.2)
- removed the REF** at (209.1, 54.8)
- added REF**: MountingHole_4.3mm_M4_DIN965_Pad, MountingHole:MountingHole_4.3mm_M4_DIN965_Pad, F.Cu at (57.0, 55.0)
- added REF**: MountingHole_4.3mm_M4_DIN965_Pad, MountingHole:MountingHole_4.3mm_M4_DIN965_Pad, F.Cu at (206.8, 55.0)
- added REF**: MountingHole_4.3mm_M4_DIN965_Pad, MountingHole:MountingHole_4.3mm_M4_DIN965_Pad, F.Cu at (57.0, 129.0)
- added REF**: MountingHole_4.3mm_M4_DIN965_Pad, MountingHole:MountingHole_4.3mm_M4_DIN965_Pad, F.Cu at (242.0, 129.0)
Other:
- board text added: "leadedsolder.com 2024, version 2"
- board text removed: "TODO: measure mounting holes"
- board text removed: "leadedsolder.com 2024, version 1"
