File: pc6001-meanwell-psu-adapter.kicad_pcb (KiCad board)
At the start: 2 copper layers, 195 x 84 mm, 5 parts, among them J1 Meanwell RPT-60B PSU module

Commit message: V2 to fab
Parts:
- moved REF** 12.2 mm to (229.8, 128.8)
- moved REF** 0.28 mm to (57.2, 128.8)
- moved REF** 0.20 mm to (57.2, 55.0)
Changed lines of the file:
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@@
 			(drillshape 0)
 			(scaleselection 1)
-			(outputdirectory "pc6001-rpt60b-v1")
+			(outputdirectory "pc6001-rpt60b-v2")
 		)
 	)
@@
 	(footprint "MountingHole:MountingHole_4.3mm_M4_DIN965_Pad"
 		(layer "F.Cu")
-		(at 57 55)
+		(at 57.2 55)
 		(descr "Mounting Hole 4.3mm, M4, DIN965")
 		(tags "mounting hole 4.3mm m4 din965")
@@
 	(footprint "MountingHole:MountingHole_4.3mm_M4_DIN965_Pad"
 		(layer "F.Cu")
-		(at 57 129)
+		(at 57.2 128.8)
 		(descr "Mounting Hole 4.3mm, M4, DIN965")
 		(tags "mounting hole 4.3mm m4 din965")
@@
 	(footprint "MountingHole:MountingHole_4.3mm_M4_DIN965_Pad"
 		(layer "F.Cu")
-		(at 242 129)
+		(at 229.8 128.8)
 		(descr "Mounting Hole 4.3mm, M4, DIN965")
 		(tags "mounting hole 4.3mm m4 din965")
@@
 		(layer "Cmts.User")
 		(pts
-			(xy 52 50) (xy 54.8 50)
-		)
-		(height 112.2)
-		(gr_text "2.8000 mm"
-			(at 53.4 161.05 0)
+			(xy 59.15 55) (xy 204.65 54.9)
+		)
+		(height -11.107854)
+		(gr_text "145.5000 mm"
+			(at 131.891576 42.692149 0.03937853642)
 			(layer "Cmts.User")
 			(effects
@@
 		(layer "Cmts.User")
 		(pts
-			(xy 59.15 55) (xy 204.65 54.9)
-		)
-		(height -11.107854)
-		(gr_text "145.5000 mm"
-			(at 131.891576 42.692149 0.03937853642)
+			(xy 52 134) (xy 55 134)
+		)
+		(height -95.5)
+		(gr_text "3.0000 mm"
+			(at 53.5 37.35 0)
 			(layer "Cmts.User")
 			(effects
@@
 		(layer "Cmts.User")
 		(pts
-			(xy 247 134) (xy 244.2 134)
-		)
-		(height 105)
-		(gr_text "2.8000 mm"
-			(at 245.6 27.85 0)
+			(xy 247 134) (xy 232 134)
+		)
+		(height 109)
+		(gr_text "15.0000 mm"
+			(at 239.5 23.85 0)
 			(layer "Cmts.User")
 			(effects
@@
 		)
 		(style
-			(thickness 0.15)
+			(thickness 0.1)
 			(arrow_length 1.27)
 			(text_position_mode 0)
@@
 		(layer "Cmts.User")
 		(pts
-			(xy 52 134) (xy 52 131.2)
-		)
-		(height 215)
-		(gr_text "2.8000 mm"
-			(at 265.85 132.6 90)
+			(xy 52 134) (xy 52 131)
+		)
+		(height 224.5)
+		(gr_text "3.0000 mm"
+			(at 275.35 132.5 90)
 			(layer "Cmts.User")
 			(effects
@@
 		)
 		(style
-			(thickness 0.15)
+			(thickness 0.1)
 			(arrow_length 1.27)
 			(text_position_mode 0)
